Commit message: Support configurable ACT and SmolVLA policy deployment
Add policy CLI arguments for checkpoint/dataset/type selection, handle ACT vs SmolVLA camera renaming, make CUDA policy multiprocessing spawn-safe, and document the updated deployment workflow.

File: URDF/Piper/collision_space_single_arm.urdf (robot description, URDF)
Before this commit: robot collision_space_single_arm, 8 links, 7 joints
Links:
- removed link left_wall
- removed link right_wall
Joints:
- removed joint world_to_left_wall
- removed joint world_to_right_wall
